File: hardware/kicad/mini-pov-wifi.kicad_sch (KiCad schematic)
At the start: 0 parts

Commit message: Fix KiCad schematic syntax for effects and hide properties.
Co-authored-by: Cursor <cursoragent@cursor.com>
Other:
- note added: "MiniPOV WiFi - Blockschaltbild (Skizze). Verdrahtung: BT1 2xAA -> U1 MT3608 -> +5V; J2 USB-C -> +5V; U2 Wemos; 8x LED mit 100R. Details in docs/HARDWARE.md"
- note removed: "MiniPOV WiFi – Blockschaltbild (Skizze) Verdrahtung: BT1 2xAA → U1 MT3608 (IN+/IN-) → OUT+ via D9 Schottky → +5V J2 USB-C VBUS via D10 Schottky → +5V +5V → U2 Wemos 5V GND gemeinsam U2 D1→R1→D1 LED, D2→R2→D2 … D0→R8→D8 (GPIO→100R→Anode, Kathode→GND) Footprints & Platzierung siehe PCB. D9/D10: Device:D_Schottky (1N5817) C1: 100µF, C2: 100nF nahe U2/U1"
Changed lines of the file:
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@@
 (kicad_sch
   (version 20231120)
-  (generator "mini-pov-wifi")
+  (generator "eeschema")
+  (generator_version "8.0")
   (paper "A3")
   (title_block
@@
     (rev "0.1")
     (company "Open Hardware")
-    (comment 1 "ESP8266 POV – 2xAA + USB-C")
+    (comment 1 "ESP8266 POV - 2xAA + USB-C")
     (comment 2 "See docs/HARDWARE.md for full wiring")
-    (comment 3 "PCB layout: hardware/kicad/mini-pov-wifi.kicad_pcb")
-    (comment 4 "Assign footprints from mini-pov-wifi.pretty")
+    (comment 3 "PCB: hardware/kicad/mini-pov-wifi.kicad_pcb")
+    (comment 4 "Footprints: mini-pov-wifi.pretty")
   )
-  (text "MiniPOV WiFi – Blockschaltbild (Skizze)\n\nVerdrahtung:\n  BT1 2xAA → U1 MT3608 (IN+/IN-) → OUT+ via D9 Schottky → +5V\n  J2 USB-C VBUS via D10 Schottky → +5V\n  +5V → U2 Wemos 5V\n  GND gemeinsam\n\n  U2 D1→R1→D1 LED, D2→R2→D2 … D0→R8→D8\n  (GPIO→100R→Anode, Kathode→GND)\n\nFootprints & Platzierung siehe PCB.\nD9/D10: Device:D_Schottky (1N5817)\nC1: 100µF, C2: 100nF nahe U2/U1"
-    (exclude_from_sim no) (at 25.4 25.4 0) (effects (font (size 2.5 2.5) (thickness 0.3) bold no italic no)))
-  (symbol (lib_id "mini-pov-wifi:Power_5V") (at 50.8 50.8 0) (unit 1) (exclude_from_sim no) (in_bom yes) (on_board yes) (dnp no)
-    (property "Reference" "#PWR01" (at 50.8 48.26 0) (effects (font (size 1.27 1.27)) hide yes))
-    (property "Value" "5V" (at 50.8 45.72 0) (effects (font (size 1.27 1.27))))
-    (pin "1")
+  (text "MiniPOV WiFi - Blockschaltbild (Skizze). Verdrahtung: BT1 2xAA -> U1 MT3608 -> +5V; J2 USB-C -> +5V; U2 Wemos; 8x LED mit 100R. Details in docs/HARDWARE.md"
+    (exclude_from_sim no)
+    (at 25.4 25.4 0)
+    (effects
+      (font (size 2.5 2.5) (thickness 0.3))
+      (justify left top)
+    )
   )
-  (symbol (lib_id "mini-pov-wifi:GND") (at 76.2 50.8 0) (unit 1) (exclude_from_sim no) (in_bom yes) (on_board yes) (dnp no)
-    (property "Reference" "#PWR02" (at 76.2 48.26 0) (effects (font (size 1.27 1.27)) hide yes))
-    (property "Value" "GND" (at 76.2 45.72 0) (effects (font (size 1.27 1.27))))
-    (pin "1")
+  (symbol
+    (lib_id "mini-pov-wifi:Power_5V")
+    (at 50.8 50.8 0)
+    (unit 1)
+    (exclude_from_sim no)
+    (in_bom yes)
+    (on_board yes)
+    (dnp no)
+    (fields_autoplaced yes)
+    (property "Reference" "#PWR01"
+      (at 50.8 48.26 0)
+      (effects
+        (font (size 1.27 1.27))
+        (hide yes)
+      )
+    )
+    (property "Value" "5V"
+      (at 50.8 45.72 0)
+      (effects
+        (font (size 1.27 1.27))
+      )
+    )
+    (pin "1"
+    )
+  )
+  (symbol
+    (lib_id "mini-pov-wifi:GND")
+    (at 76.2 50.8 0)
+    (unit 1)
+    (exclude_from_sim no)
+    (in_bom yes)
+    (on_board yes)
+    (dnp no)
+    (fields_autoplaced yes)
+    (property "Reference" "#PWR02"
+      (at 76.2 48.26 0)
+      (effects
+        (font (size 1.27 1.27))
+        (hide yes)
+      )
+    )
+    (property "Value" "GND"
+      (at 76.2 45.72 0)
+      (effects
+        (font (size 1.27 1.27))
+      )
+    )
+    (pin "1"
+    )
   )
   (sheet_instances
-    (path "/" (page "1"))
+    (path "/"
+      (page "1")
+    )
   )
 )

Commit message: Fix KiCad PCB hide syntax and expand schematic with standard symbols.
Co-authored-by: Cursor <cursoragent@cursor.com>
Parts:
- added BT1: 2xAA, mini-pov-wifi:Battery_2xAA, symbol Device:Battery_Cell
- added C1: 100uF, Capacitor_THT:CP_Radial_D5.0mm_P2.50mm, symbol Device:C
- added C2: 100nF, Capacitor_THT:C_Disc_D3.0mm_W1.6mm_P2.50mm, symbol Device:C
- added D1: LED, mini-pov-wifi:LED_D5.0mm, symbol Device:LED
- added D10, D9: 1N5817, Diode_THT:D_DO-41_SOD81_P10.16mm_Horizontal, symbol Device:D_Schottky
- added R1: 100R, mini-pov-wifi:R_THT_1-4W, symbol Device:R
- added U2: Wemos_D1_Mini, mini-pov-wifi:Wemos_D1_Mini_Socket, symbol Connector_Generic:Conn_02x08_Odd_Even
Other:
- note added: "J2 footprint: mini-pov-wifi:USB-C_Breakout"
- note added: "Power: 2xAA -> MT3608 U1 -> +5V rail. USB-C J2 -> Schottky D10 -> +5V. Wemos U2 on 5V/GND. GPIO -> 100R -> LED -> GND."
- note added: "R2-R8 / D2-D8: same chain (see PCB). U1 MT3608 module: IN+ IN- OUT+ OUT-. J2 USB-C breakout: VBUS GND."
- note added: "U1 footprint: mini-pov-wifi:MT3608_Module"
- note removed: "MiniPOV WiFi - Blockschaltbild (Skizze). Verdrahtung: BT1 2xAA -> U1 MT3608 -> +5V; J2 USB-C -> +5V; U2 Wemos; 8x LED mit 100R. Details in docs/HARDWARE.md"
- title: MiniPOV WiFi -> ESPOV / MiniPOV WiFi
Changed lines of the file:
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@@
   (paper "A3")
   (title_block
-    (title "MiniPOV WiFi")
+    (title "ESPOV / MiniPOV WiFi")
     (date "2026-07-22")
-    (rev "0.1")
+    (rev "0.2")
     (company "Open Hardware")
-    (comment 1 "ESP8266 POV - 2xAA + USB-C")
-    (comment 2 "See docs/HARDWARE.md for full wiring")
-    (comment 3 "PCB: hardware/kicad/mini-pov-wifi.kicad_pcb")
-    (comment 4 "Footprints: mini-pov-wifi.pretty")
+    (comment 1 "ESP8266 POV - 2xAA + Boost + USB-C")
+    (comment 2 "Footprints: hardware/kicad/mini-pov-wifi.pretty")
+    (comment 3 "Details: docs/HARDWARE.md")
+    (comment 4 "Assign footprints after opening in KiCad")
   )
-  (text "MiniPOV WiFi - Blockschaltbild (Skizze). Verdrahtung: BT1 2xAA -> U1 MT3608 -> +5V; J2 USB-C -> +5V; U2 Wemos; 8x LED mit 100R. Details in docs/HARDWARE.md"
+  (text "Power: 2xAA -> MT3608 U1 -> +5V rail. USB-C J2 -> Schottky D10 -> +5V. Wemos U2 on 5V/GND. GPIO -> 100R -> LED -> GND."
     (exclude_from_sim no)
-    (at 25.4 25.4 0)
-    (effects
-      (font (size 2.5 2.5) (thickness 0.3))
-      (justify left top)
-    )
+    (at 20.32 20.32 0)
+    (effects (font (size 1.8 1.8) (thickness 0.25)) (justify left top))
   )
-  (symbol
-    (lib_id "mini-pov-wifi:Power_5V")
-    (at 50.8 50.8 0)
-    (unit 1)
+  (symbol (lib_id "power:+5V") (at 50.8 40.64 0) (unit 1)
+    (exclude_from_sim no) (in_bom yes) (on_board yes) (dnp no)
+    (property "Reference" "#PWR01" (at 50.8 36.83 0) (effects (font (size 1.27 1.27)) (hide yes)))
+    (property "Value" "+5V" (at 50.8 38.1 0) (effects (font (size 1.27 1.27))))
+    (pin "1")
+  )
+  (symbol (lib_id "power:+5V") (at 127 40.64 0) (unit 1)
+    (exclude_from_sim no) (in_bom yes) (on_board yes) (dnp no)
+    (property "Reference" "#PWR02" (at 127 36.83 0) (effects (font (size 1.27 1.27)) (hide yes)))
+    (property "Value" "+5V" (at 127 38.1 0) (effects (font (size 1.27 1.27))))
+    (pin "1")
+  )
+  (symbol (lib_id "power:GND") (at 50.8 175.26 0) (unit 1)
+    (exclude_from_sim no) (in_bom yes) (on_board yes) (dnp no)
+    (property "Reference" "#PWR03" (at 50.8 181.61 0) (effects (font (size 1.27 1.27)) (hide yes)))
+    (property "Value" "GND" (at 50.8 179.07 0) (effects (font (size 1.27 1.27))))
+    (pin "1")
+  )
+  (symbol (lib_id "power:GND") (at 127 175.26 0) (unit 1)
+    (exclude_from_sim no) (in_bom yes) (on_board yes) (dnp no)
+    (property "Reference" "#PWR04" (at 127 181.61 0) (effects (font (size 1.27 1.27)) (hide yes)))
+    (property "Value" "GND" (at 127 179.07 0) (effects (font (size 1.27 1.27))))
+    (pin "1")
+  )
+  (symbol (lib_id "Device:Battery_Cell") (at 30.48 68.58 0) (unit 1)
+    (exclude_from_sim no) (in_bom yes) (on_board yes) (dnp no)
+    (property "Reference" "BT1" (at 33.02 67.31 0) (effects (font (size 1.27 1.27)) (justify left)))
+    (property "Value" "2xAA" (at 33.02 69.85 0) (effects (font (size 1.27 1.27)) (justify left)))
+    (property "Footprint" "mini-pov-wifi:Battery_2xAA" (at 30.48 68.58 0) (effects (font (size 1.27 1.27)) (hide yes)))
+    (pin "1")
+    (pin "2")
+  )
+  (symbol (lib_id "Device:D_Schottky") (at 76.2 50.8 0) (unit 1)
+    (exclude_from_sim no) (in_bom yes) (on_board yes) (dnp no)
+    (property "Reference" "D9" (at 79.375 49.53 0) (effects (font (size 1.27 1.27)) (justify left)))
+    (property "Value" "1N5817" (at 79.375 52.07 0) (effects (font (size 1.27 1.27)) (justify left)))
+    (property "Footprint" "Diode_THT:D_DO-41_SOD81_P10.16mm_Horizontal" (at 76.2 50.8 0) (effects (font (size 1.27 1.27)) (hide yes)))
+    (pin "1")
+    (pin "2")
+  )
+  (symbol (lib_id "Device:D_Schottky") (at 101.6 50.8 0) (unit 1)
+    (exclude_from_sim no) (in_bom yes) (on_board yes) (dnp no)
+    (property "Reference" "D10" (at 104.775 49.53 0) (effects (font (size 1.27 1.27)) (justify left)))
+    (property "Value" "1N5817" (at 104.775 52.07 0) (effects (font (size 1.27 1.27)) (justify left)))
+    (property "Footprint" "Diode_THT:D_DO-41_SOD81_P10.16mm_Horizontal" (at 101.6 50.8 0) (effects (font (size 1.27 1.27)) (hide yes)))
+    (pin "1")
+    (pin "2")
+  )
+  (symbol (lib_id "Device:C") (at 88.9 63.5 0) (unit 1)
+    (exclude_from_sim no) (in_bom yes) (on_board yes) (dnp no)
+    (property "Reference" "C1" (at 91.44 62.23 0) (effects (font (size 1.27 1.27)) (justify left)))
+    (property "Value" "100uF" (at 91.44 64.77 0) (effects (font (size 1.27 1.27)) (justify left)))
+    (property "Footprint" "Capacitor_THT:CP_Radial_D5.0mm_P2.50mm" (at 88.9 63.5 0) (effects (font (size 1.27 1.27)) (hide yes)))
+    (pin "1")
+    (pin "2")
+  )
+  (symbol (lib_id "Device:C") (at 114.3 88.9 0) (unit 1)
+    (exclude_from_sim no) (in_bom yes) (on_board yes) (dnp no)
+    (property "Reference" "C2" (at 116.84 87.63 0) (effects (font (size 1.27 1.27)) (justify left)))
+    (property "Value" "100nF" (at 116.84 90.17 0) (effects (font (size 1.27 1.27)) (justify left)))
+    (property "Footprint" "Capacitor_THT:C_Disc_D3.0mm_W1.6mm_P2.50mm" (at 114.3 88.9 0) (effects (font (size 1.27 1.27)) (hide yes)))
+    (pin "1")
+    (pin "2")
+  )
+  (symbol (lib_id "Connector_Generic:Conn_02x08_Odd_Even") (at 88.9 114.3 0) (unit 1)
+    (exclude_from_sim no) (in_bom yes) (on_board yes) (dnp no)
+    (property "Reference" "U2" (at 88.9 99.06 0) (effects (font (size 1.27 1.27))))
+    (property "Value" "Wemos_D1_Mini" (at 88.9 129.54 0) (effects (font (size 1.27 1.27))))
+    (property "Footprint" "mini-pov-wifi:Wemos_D1_Mini_Socket" (at 88.9 114.3 0) (effects (font (size 1.27 1.27)) (hide yes)))
+    (pin "1")
+    (pin "2")
+    (pin "3")
+    (pin "4")
+    (pin "5")
+    (pin "6")
+    (pin "7")
+    (pin "8")
+    (pin "9")
+    (pin "10")
+    (pin "11")
+    (pin "12")
+    (pin "13")
+    (pin "14")
+    (pin "15")
+    (pin "16")
+  )
+  (symbol (lib_id "Device:R") (at 152.4 88.9 0) (unit 1)
+    (exclude_from_sim no) (in_bom yes) (on_board yes) (dnp no)
+    (property "Reference" "R1" (at 154.94 87.63 0) (effects (font (size 1.27 1.27)) (justify left)))
+    (property "Value" "100R" (at 154.94 90.17 0) (effects (font (size 1.27 1.27)) (justify left)))
+    (property "Footprint" "mini-pov-wifi:R_THT_1-4W" (at 152.4 88.9 0) (effects (font (size 1.27 1.27)) (hide yes)))
+    (pin "1")
+    (pin "2")
+  )
+  (symbol (lib_id "Device:LED") (at 177.8 88.9 0) (unit 1)
+    (exclude_from_sim no) (in_bom yes) (on_board yes) (dnp no)
+    (property "Reference" "D1" (at 180.34 87.63 0) (effects (font (size 1.27 1.27)) (justify left)))
+    (property "Value" "LED" (at 180.34 90.17 0) (effects (font (size 1.27 1.27)) (justify left)))
+    (property "Footprint" "mini-pov-wifi:LED_D5.0mm" (at 177.8 88.9 0) (effects (font (size 1.27 1.27)) (hide yes)))
+    (pin "1")
+    (pin "2")
+  )
+  (text "R2-R8 / D2-D8: same chain (see PCB). U1 MT3608 module: IN+ IN- OUT+ OUT-. J2 USB-C breakout: VBUS GND."
     (exclude_from_sim no)
-    (in_bom yes)
-    (on_board yes)
-    (dnp no)
-    (fields_autoplaced yes)
-    (property "Reference" "#PWR01"
-      (at 50.8 48.26 0)
-      (effects
-        (font (size 1.27 1.27))
-        (hide yes)
-      )
-    )
-    (property "Value" "5V"
-      (at 50.8 45.72 0)
-      (effects
-        (font (size 1.27 1.27))
-      )
-    )
-    (pin "1"
-    )
+    (at 20.32 139.7 0)
+    (effects (font (size 1.5 1.5) (thickness 0.2)) (justify left top))
   )
-  (symbol
-    (lib_id "mini-pov-wifi:GND")
-    (at 76.2 50.8 0)
-    (unit 1)
+  (text "U1 footprint: mini-pov-wifi:MT3608_Module"
     (exclude_from_sim no)
-    (in_bom yes)
-    (on_board yes)
-    (dnp no)
-    (fields_autoplaced yes)
-    (property "Reference" "#PWR02"
-      (at 76.2 48.26 0)
-      (effects
-        (font (size 1.27 1.27))
-        (hide yes)
-      )
-    )
-    (property "Value" "GND"
-      (at 76.2 45.72 0)
-      (effects
-        (font (size 1.27 1.27))
-      )
-    )
-    (pin "1"
-    )
+    (at 55.88 50.8 0)
+    (effects (font (size 1.27 1.27) (thickness 0.15)) (justify left))
   )
-  (sheet_instances
-    (path "/"
-      (page "1")
-    )
+  (text "J2 footprint: mini-pov-wifi:USB-C_Breakout"
+    (exclude_from_sim no)
+    (at 81.28 50.8 0)
+    (effects (font (size 1.27 1.27) (thickness 0.15)) (justify left))
   )
+  (wire (pts (xy 50.8 44.45) (xy 50.8 50.8)) (stroke (width 0) (type default)))
+  (wire (pts (xy 127 44.45) (xy 127 50.8)) (stroke (width 0) (type default)))
+  (wire (pts (xy 50.8 50.8) (xy 73.66 50.8)) (stroke (width 0) (type default)))
+  (wire (pts (xy 78.74 50.8) (xy 127 50.8)) (stroke (width 0) (type default)))
+  (wire (pts (xy 50.8 175.26) (xy 50.8 170.18)) (stroke (width 0) (type default)))
+  (wire (pts (xy 127 175.26) (xy 127 170.18)) (stroke (width 0) (type default)))
+  (wire (pts (xy 33.02 68.58) (xy 45.72 68.58)) (stroke (width 0) (type default)))
+  (wire (pts (xy 33.02 73.66) (xy 45.72 73.66)) (stroke (width 0) (type default)))
+  (wire (pts (xy 50.8 170.18) (xy 127 170.18)) (stroke (width 0) (type default)))
+  (wire (pts (xy 154.94 88.9) (xy 175.26 88.9)) (stroke (width 0) (type default)))
+  (wire (pts (xy 180.34 88.9) (xy 190.5 88.9)) (stroke (width 0) (type default)))
+  (wire (pts (xy 190.5 88.9) (xy 190.5 170.18)) (stroke (width 0) (type default)))
+  (label "BAT+" (at 45.72 68.58 0) (fields_autoplaced yes)
+    (effects (font (size 1.27 1.27)) (justify right bottom))
+  )
+  (label "BAT-" (at 45.72 73.66 0) (fields_autoplaced yes)
+    (effects (font (size 1.27 1.27)) (justify right bottom))
+  )
+  (label "LED1" (at 149.86 88.9 0) (fields_autoplaced yes)
+    (effects (font (size 1.27 1.27)) (justify right bottom))
+  )
+  (sheet_instances (path "/" (page "1")))
 )

Commit message: Rebuild schematic: power, Wemos, and full 8-LED array with embedded symbols.
Co-authored-by: Cursor <cursoragent@cursor.com>
Parts:
- removed BT1: 2xAA, mini-pov-wifi:Battery_2xAA, symbol Device:Battery_Cell
- removed U2: Wemos_D1_Mini, mini-pov-wifi:Wemos_D1_Mini_Socket, symbol Connector_Generic:Conn_02x08_Odd_Even
- added BT1: 2xAA, mini-pov-wifi:Battery_2xAA, symbol Device:Battery
- added D2, D3, D4, D5, D6, D7, D8: LED, mini-pov-wifi:LED_D5.0mm, symbol Device:LED
- added J2: USB-C, mini-pov-wifi:USB-C_Breakout, symbol Connector:Conn_01x02
- added R2, R3, R4, R5, R6, R7, R8: 100R, mini-pov-wifi:R_THT_1-4W, symbol Device:R
- added U1: MT3608, mini-pov-wifi:MT3608_Module, symbol Connector:Conn_01x04
- added U2: Wemos D1 Mini, mini-pov-wifi:Wemos_D1_Mini_Socket, symbol espov:Wemos_D1_Mini
- C2: footprint Capacitor_THT:C_Disc_D3.0mm_W1.6mm_P2.50mm -> (none)
Connections:
- new net: R1.1, R2.1, R3.1, R4.1, R5.1, R6.1, R7.1, R8.1, U2.10 (MOSI), U2.20 (A0), U2.9 (MISO)
- new net: D6.2 (A), R6.2
- new net: D10.2 (A), J2.2
- new net: D4.2 (A), R4.2
- new net: D3.2 (A), R3.2
- new net: D5.2 (A), R5.2
- new net: D7.2 (A), R7.2
- new net: D1.2 (A), R1.2
- new net: D9.2 (A), U1.2
- new net: D2.2 (A), R2.2
- new net: D8.2 (A), R8.2
- new net +5V: BT1.1 (+), BT1.2 (-), C1.1, C1.2, C2.1, C2.2, D1.1 (K), D10.1 (K), D2.1 (K), D3.1 (K), D4.1 (K), D5.1 (K), D6.1 (K), D7.1 (K), D8.1 (K), D9.1 (K), J2.1, U1.1, U1.3, U1.4
- no-connect marks 0 -> 9
Other:
- note added: "1. Power"
- note added: "2. Controller"
- note added: "3. POV LEDs"
- note added: "D3/FLASH = WiFi config button (on module)"
- note added: "D9/D10 = Schottky OR (Boost + USB -> +5V)"
- note added: "GPIO -> 100R -> LED Anode; Kathode -> GND"
- note removed: "J2 footprint: mini-pov-wifi:USB-C_Breakout"
- note removed: "Power: 2xAA -> MT3608 U1 -> +5V rail. USB-C J2 -> Schottky D10 -> +5V. Wemos U2 on 5V/GND. GPIO -> 100R -> LED -> GND."
- note removed: "R2-R8 / D2-D8: same chain (see PCB). U1 MT3608 module: IN+ IN- OUT+ OUT-. J2 USB-C breakout: VBUS GND."
- note removed: "U1 footprint: mini-pov-wifi:MT3608_Module"
- company: Open Hardware -> (none)
- title: ESPOV / MiniPOV WiFi -> ESPOV - MiniPOV WiFi
